Commit message: Update robot.xacro
change wheel frame

File: robot_description/urdf/robot.xacro (robot description, xacro)
@@ -22,4 +22,5 @@
   <link name="front_wheel">
     <visual>
+      <origin xyz="0 0 0" rpy="${pi/2} 0 0"/>
       <geometry>
         <cylinder radius="0.031" length="0.025"/>
@@ -27,4 +28,5 @@
     </visual>
     <collision>
+      <origin xyz="0 0 0" rpy="${pi/2} 0 0"/>
       <geometry>
         <cylinder radius="0.031" length="0.025"/>
@@ -39,11 +41,12 @@
     <parent link="chassis"/>
     <child link="front_wheel"/>
-    <origin xyz="0.16 0.0 -0.06" rpy="${3.14/2} 0 0"/>
-    <axis xyz="0 0 1"/>
-    <limit effort="100" velocity="3.0"/>
+    <origin xyz="0.16 0.0 -0.06" rpy="0 0 0"/>
+    <axis xyz="0 1 0"/>
+    <limit effort="100" velocity="2.5"/>
   </joint>
   <!-- Rear Left Wheel -->
   <link name="rear_left_wheel">
     <visual>
+      <origin xyz="0 0 0" rpy="${pi/2} 0 0"/>
       <geometry>
         <cylinder radius="0.031" length="0.025"/>
@@ -51,4 +54,5 @@
     </visual>
     <collision>
+      <origin xyz="0 0 0" rpy="${pi/2} 0 0"/>
       <geometry>
         <cylinder radius="0.031" length="0.025"/>
@@ -63,11 +67,12 @@
     <parent link="chassis"/>
     <child link="rear_left_wheel"/>
-    <origin xyz="-0.16 0.08 -0.06" rpy="${3.14/2} 0 0"/>
-    <axis xyz="0 0 1"/>
-    <limit effort="100" velocity="3.0"/>
+    <origin xyz="-0.16 0.08 -0.06" rpy="0 0 0"/>
+    <axis xyz="0 1 0"/>
+    <limit effort="100" velocity="2.5"/>
   </joint>
   <!-- Rear Right Wheel -->
   <link name="rear_right_wheel">
     <visual>
+      <origin xyz="0 0 0" rpy="${pi/2} 0 0"/>
       <geometry>
         <cylinder radius="0.031" length="0.025"/>
@@ -75,4 +80,5 @@
     </visual>
     <collision>
+      <origin xyz="0 0 0" rpy="${pi/2} 0 0"/>
       <geometry>
         <cylinder radius="0.031" length="0.025"/>
@@ -87,6 +93,6 @@
     <parent link="chassis"/>
     <child link="rear_right_wheel"/>
-    <origin xyz="-0.16 -0.08 -0.06" rpy="${3.14/2} 0 0"/>
-    <axis xyz="0 0 1"/>
+    <origin xyz="-0.16 -0.08 -0.06" rpy="0 0 0"/>
+    <axis xyz="0 1 0"/>
     <limit effort="100" velocity="3.0"/>
   </joint>

Commit message: change front wheel joint to revolute

File: robot_description/urdf/robot.xacro (robot description, xacro)
@@ -38,10 +38,10 @@
   </link>
   <!-- Front Wheel Joint -->
-  <joint name="front_wheel_joint" type="continuous">
+  <joint name="front_wheel_joint" type="revolute">
     <parent link="chassis"/>
     <child link="front_wheel"/>
     <origin xyz="0.16 0.0 -0.06" rpy="0 0 0"/>
-    <axis xyz="0 1 0"/>
-    <limit effort="10.0" velocity="3.0"/>
+    <axis xyz="0 0 1"/>
+    <limit lower="-0.698" upper="0.698" effort="10.0" velocity="3.0"/>
   </joint>
   <!-- Rear Left Wheel -->
