Commit message: update robot.xacro

File: robot_description/urdf/gazebo.xacro (robot description, xacro)
@@ -6,5 +6,5 @@
             <plugin>gazebo_ros2_control/GazeboSystem</plugin>
         </hardware>
-        <joint name="joint_1">
+        <joint name="front_wheel_joint">
             <command_interface name="position">
                 <param name="min">-3.14</param>
@@ -18,5 +18,5 @@
             <state_interface name="effort"/>
         </joint>
-        <joint name="joint_2">
+        <joint name="rear_left_wheel_joint">
             <command_interface name="velocity"/>
             <command_interface name="position">
@@ -30,5 +30,5 @@
             <state_interface name="effort"/>
         </joint>
-        <joint name="joint_3">
+        <joint name="rear_right_wheel_joint">
             <command_interface name="velocity"/>
             <command_interface name="position">
@@ -49,20 +49,20 @@
         </plugin>
     </gazebo>
-    <gazebo reference="link_0">
+    <gazebo reference="chassis">
         <mu1>0.2</mu1>
         <mu2>0.2</mu2>
         <material>Gazebo/Green</material>
     </gazebo>
-    <gazebo reference="link_1">
+    <gazebo reference="front_wheel">
         <mu1>0.2</mu1>
         <mu2>0.2</mu2>
         <material>Gazebo/Red</material>
     </gazebo>
-    <gazebo reference="link_2">
+    <gazebo reference="rear_left_wheel">
         <mu1>0.2</mu1>
         <mu2>0.2</mu2>
         <material>Gazebo/Blue</material>
     </gazebo>
-    <gazebo reference="link_3">
+    <gazebo reference="rear_right_wheel">
         <mu1>0.2</mu1>
         <mu2>0.2</mu2>

File: robot_description/urdf/robot.xacro (robot description, xacro)
@@ -34,4 +34,12 @@
     </xacro:inertial_cylinder>
   </link>
+  <!-- Front Wheel Joint -->
+  <joint name="front_wheel_joint" type="revolute">
+    <parent link="chassis"/>
+    <child link="front_wheel"/>
+    <origin xyz="0.16 0.0 -0.0155" rpy="${3.14/2} 0 0"/>
+    <axis xyz="1 0 0"/>
+    <limit lower="-3.14" upper="3.14" effort="100" velocity="10"/>
+  </joint>
   <!-- Rear Left Wheel -->
   <link name="rear_left_wheel">
@@ -50,4 +58,12 @@
     </xacro:inertial_cylinder>
   </link>
+   <!-- Rear Left Wheel Joint -->
+  <joint name="rear_left_wheel_joint" type="revolute">
+    <parent link="chassis"/>
+    <child link="rear_left_wheel"/>
+    <origin xyz="-0.16 0.08 -0.0155" rpy="${3.14/2} 0 0"/>
+    <axis xyz="1 0 0"/>
+    <limit lower="-3.14" upper="3.14" effort="100" velocity="10"/>
+  </joint>
   <!-- Rear Right Wheel -->
   <link name="rear_right_wheel">
@@ -66,20 +82,4 @@
     </xacro:inertial_cylinder>
   </link>
-  <!-- Front Wheel Joint -->
-  <joint name="front_wheel_joint" type="revolute">
-    <parent link="chassis"/>
-    <child link="front_wheel"/>
-    <origin xyz="0.16 0.0 -0.0155" rpy="${3.14/2} 0 0"/>
-    <axis xyz="1 0 0"/>
-    <limit lower="-3.14" upper="3.14" effort="100" velocity="10"/>
-  </joint>
-  <!-- Rear Left Wheel Joint -->
-  <joint name="rear_left_wheel_joint" type="revolute">
-    <parent link="chassis"/>
-    <child link="rear_left_wheel"/>
-    <origin xyz="-0.16 0.08 -0.0155" rpy="${3.14/2} 0 0"/>
-    <axis xyz="1 0 0"/>
-    <limit lower="-3.14" upper="3.14" effort="100" velocity="10"/>
-  </joint>
   <!-- Rear Right Wheel Joint -->
   <joint name="rear_right_wheel_joint" type="revolute">

Commit message: spawn robot in gazebo

File: robot_description/urdf/gazebo.xacro (robot description, xacro)
@@ -1,5 +1,4 @@
 <?xml version="1.0"?>
-<robot xmlns:xacro="http://www.ros.org/wiki/xacro" name="example">
-    <xacro:include filename="inertial_macros.xacro"/>
+<robot xmlns:xacro="http://www.ros.org/wiki/xacro" name="f1tenth">
     <ros2_control name="GazeboSystem" type="system">
         <hardware>
@@ -7,8 +6,4 @@
         </hardware>
         <joint name="front_wheel_joint">
-            <command_interface name="position">
-                <param name="min">-3.14</param>
-                <param name="max">3.14</param>
-            </command_interface>
             <command_interface name="velocity"/>
             <state_interface name="position">
@@ -20,8 +15,4 @@
         <joint name="rear_left_wheel_joint">
             <command_interface name="velocity"/>
-            <command_interface name="position">
-                <param name="min">-3.14</param>
-                <param name="max">3.14</param>
-            </command_interface>
             <state_interface name="position">
                 <param name="initial_value">0.0</param>
@@ -32,8 +23,4 @@
         <joint name="rear_right_wheel_joint">
             <command_interface name="velocity"/>
-            <command_interface name="position">
-                <param name="min">-3.14</param>
-                <param name="max">3.14</param>
-            </command_interface>
             <state_interface name="position">
                 <param name="initial_value">0.0</param>
@@ -46,25 +33,25 @@
         <plugin filename="libgazebo_ros2_control.so" name="gazebo_ros2_control">
             <robot_sim_type>gazebo_ros2_control/GazeboSystem</robot_sim_type>
-            <parameters>$(find robot_description)/config/controllers.yaml</parameters>
+            <parameters>$(find robot_description)/config/controller.yaml</parameters>
         </plugin>
     </gazebo>
     <gazebo reference="chassis">
-        <mu1>0.2</mu1>
-        <mu2>0.2</mu2>
-        <material>Gazebo/Green</material>
+        <mu1>1.0</mu1>
+        <mu2>1.0</mu2>
+        <material>Gazebo/White</material>
     </gazebo>
     <gazebo reference="front_wheel">
-        <mu1>0.2</mu1>
-        <mu2>0.2</mu2>
-        <material>Gazebo/Red</material>
+        <mu1>1.0</mu1>
+        <mu2>1.0</mu2>
+        <material>Gazebo/Black</material>
     </gazebo>
     <gazebo reference="rear_left_wheel">
-        <mu1>0.2</mu1>
-        <mu2>0.2</mu2>
-        <material>Gazebo/Blue</material>
+        <mu1>1.0</mu1>
+        <mu2>1.0</mu2>
+        <material>Gazebo/Black</material>
     </gazebo>
     <gazebo reference="rear_right_wheel">
-        <mu1>0.2</mu1>
-        <mu2>0.2</mu2>
+        <mu1>1.0</mu1>
+        <mu2>1.0</mu2>
         <material>Gazebo/Black</material>
     </gazebo>

File: robot_description/urdf/robot.xacro (robot description, xacro)
@@ -2,4 +2,5 @@
 <robot xmlns:xacro="http://www.ros.org/wiki/xacro" name="f1tenth">
   <xacro:include filename="gazebo.xacro"/>
+  <xacro:include filename="inertial_macros.xacro"/>
   <!-- Chassis Link -->
   <link name="chassis">
@@ -35,10 +36,10 @@
   </link>
   <!-- Front Wheel Joint -->
-  <joint name="front_wheel_joint" type="revolute">
+  <joint name="front_wheel_joint" type="continuous">
     <parent link="chassis"/>
     <child link="front_wheel"/>
-    <origin xyz="0.16 0.0 -0.0155" rpy="${3.14/2} 0 0"/>
-    <axis xyz="1 0 0"/>
-    <limit lower="-3.14" upper="3.14" effort="100" velocity="10"/>
+    <origin xyz="0.16 0.0 -0.06" rpy="${3.14/2} 0 0"/>
+    <axis xyz="0 0 1"/>
+    <limit effort="100" velocity="3.0"/>
   </joint>
   <!-- Rear Left Wheel -->
@@ -59,10 +60,10 @@
   </link>
    <!-- Rear Left Wheel Joint -->
-  <joint name="rear_left_wheel_joint" type="revolute">
+  <joint name="rear_left_wheel_joint" type="continuous">
     <parent link="chassis"/>
     <child link="rear_left_wheel"/>
-    <origin xyz="-0.16 0.08 -0.0155" rpy="${3.14/2} 0 0"/>
-    <axis xyz="1 0 0"/>
-    <limit lower="-3.14" upper="3.14" effort="100" velocity="10"/>
+    <origin xyz="-0.16 0.08 -0.06" rpy="${3.14/2} 0 0"/>
+    <axis xyz="0 0 1"/>
+    <limit effort="100" velocity="3.0"/>
   </joint>
   <!-- Rear Right Wheel -->
@@ -83,10 +84,10 @@
   </link>
   <!-- Rear Right Wheel Joint -->
-  <joint name="rear_right_wheel_joint" type="revolute">
+  <joint name="rear_right_wheel_joint" type="continuous">
     <parent link="chassis"/>
     <child link="rear_right_wheel"/>
-    <origin xyz="-0.16 -0.08 -0.0155" rpy="${3.14/2} 0 0"/>
-    <axis xyz="1 0 0"/>
-    <limit lower="-3.14" upper="3.14" effort="100" velocity="10"/>
+    <origin xyz="-0.16 -0.08 -0.06" rpy="${3.14/2} 0 0"/>
+    <axis xyz="0 0 1"/>
+    <limit effort="100" velocity="3.0"/>
   </joint>
 </robot>

Commit message: change to effort control

File: robot_description/urdf/gazebo.xacro (robot description, xacro)
@@ -6,5 +6,6 @@
         </hardware>
         <joint name="front_wheel_joint">
-            <command_interface name="velocity"/>
+            <command_interface name="effort"/>
+            <!-- <command_interface name="velocity"/> -->
             <state_interface name="position">
                 <param name="initial_value">0.0</param>
@@ -14,5 +15,6 @@
         </joint>
         <joint name="rear_left_wheel_joint">
-            <command_interface name="velocity"/>
+            <command_interface name="effort"/>
+            <!-- <command_interface name="velocity"/> -->
             <state_interface name="position">
                 <param name="initial_value">0.0</param>
@@ -22,5 +24,6 @@
         </joint>
         <joint name="rear_right_wheel_joint">
-            <command_interface name="velocity"/>
+            <command_interface name="effort"/>
+            <!-- <command_interface name="velocity"/> -->
             <state_interface name="position">
                 <param name="initial_value">0.0</param>
@@ -37,21 +40,21 @@
     </gazebo>
     <gazebo reference="chassis">
-        <mu1>1.0</mu1>
-        <mu2>1.0</mu2>
+        <mu1>0.1</mu1>
+        <mu2>0.1</mu2>
         <material>Gazebo/White</material>
     </gazebo>
     <gazebo reference="front_wheel">
-        <mu1>1.0</mu1>
-        <mu2>1.0</mu2>
+        <mu1>0.1</mu1>
+        <mu2>0.1</mu2>
         <material>Gazebo/Black</material>
     </gazebo>
     <gazebo reference="rear_left_wheel">
-        <mu1>1.0</mu1>
-        <mu2>1.0</mu2>
+        <mu1>0.1</mu1>
+        <mu2>0.1</mu2>
         <material>Gazebo/Black</material>
     </gazebo>
     <gazebo reference="rear_right_wheel">
-        <mu1>1.0</mu1>
-        <mu2>1.0</mu2>
+        <mu1>0.1</mu1>
+        <mu2>0.1</mu2>
         <material>Gazebo/Black</material>
     </gazebo>

File: robot_description/urdf/robot.xacro (robot description, xacro)
@@ -43,5 +43,5 @@
     <origin xyz="0.16 0.0 -0.06" rpy="0 0 0"/>
     <axis xyz="0 1 0"/>
-    <limit effort="100" velocity="2.5"/>
+    <limit effort="10.0" velocity="3.0"/>
   </joint>
   <!-- Rear Left Wheel -->
@@ -69,5 +69,5 @@
     <origin xyz="-0.16 0.08 -0.06" rpy="0 0 0"/>
     <axis xyz="0 1 0"/>
-    <limit effort="100" velocity="2.5"/>
+    <limit effort="10.0" velocity="3.0"/>
   </joint>
   <!-- Rear Right Wheel -->
@@ -95,5 +95,5 @@
     <origin xyz="-0.16 -0.08 -0.06" rpy="0 0 0"/>
     <axis xyz="0 1 0"/>
-    <limit effort="100" velocity="3.0"/>
+    <limit effort="10.0" velocity="3.0"/>
   </joint>
 </robot>

Commit message: Add steer _link

File: robot_description/urdf/gazebo.xacro (robot description, xacro)
@@ -6,5 +6,5 @@
         </hardware>
         <!-- Front Wheel (Steering) -->
-        <joint name="front_wheel_joint">
+        <joint name="steer_joint">
             <command_interface name="position"/>
             <state_interface name="position">

File: robot_description/urdf/robot.xacro (robot description, xacro)
@@ -19,4 +19,28 @@
     </xacro:inertial_box>
   </link>
+  <!-- Steer Link -->
+  <link name="steer_link">
+    <visual>
+      <geometry>
+        <box size="0.025 0.025 0.031"/>
+      </geometry>
+    </visual>
+    <collision>
+      <geometry>
+        <box size="0.025 0.025 0.031"/>
+      </geometry>
+    </collision>
+    <xacro:inertial_box mass="0.02" x="0.025" y="0.025" z="0.031">
+      <origin xyz="0.0 0.0 -0.0155" rpy="0 0 0"/>
+    </xacro:inertial_box>
+  </link>
+  <!-- Steer Joint (connects chassis to steer_link) -->
+  <joint name="steer_joint" type="revolute">
+    <parent link="chassis"/>
+    <child link="steer_link"/>
+    <origin xyz="0.16 0.0 -0.06" rpy="0 0 0"/>
+    <axis xyz="0 0 1"/>
+    <limit lower="-0.698" upper="0.698" effort="10.0" velocity="3.0"/>
+  </joint>
   <!-- Front Wheel -->
   <link name="front_wheel">
@@ -37,11 +61,10 @@
     </xacro:inertial_cylinder>
   </link>
-  <!-- Front Wheel Joint -->
-  <joint name="front_wheel_joint" type="revolute">
-    <parent link="chassis"/>
+  <!-- Front Wheel Joint (connects steer_link to front_wheel) -->
+  <joint name="front_wheel_joint" type="continuous">
+    <parent link="steer_link"/>
     <child link="front_wheel"/>
-    <origin xyz="0.16 0.0 -0.06" rpy="0 0 0"/>
-    <axis xyz="0 0 1"/>
-    <limit lower="-0.698" upper="0.698" effort="10.0" velocity="3.0"/>
+    <origin xyz="0 0 0.0" rpy="0 0 0"/>
+    <axis xyz="0 1 0"/>
   </joint>
   <!-- Rear Left Wheel -->
@@ -63,5 +86,5 @@
     </xacro:inertial_cylinder>
   </link>
-   <!-- Rear Left Wheel Joint -->
+  <!-- Rear Left Wheel Joint -->
   <joint name="rear_left_wheel_joint" type="continuous">
     <parent link="chassis"/>
